File: Simple-FC.kicad_sch (KiCad schematic)
At the start: 69 parts, among them J1 USB_C_Receptacle_USB2.0_14P, J2 Micro_SD_Card, J3 Conn_01x04, J4 Conn_01x04, J5 Conn_01x04, J6 Conn_01x05, J7 Conn_01x04, J8 Conn_01x03, SW1 SW_Push, U1 RP2350A, U2 MMC5983MA, U3 LSM6DSM, U4 BMP384, U5 TPS631000, U6 W25Q128JVS, Y1 ABM8-272-T3

Commit message: started pcb layout
Parts:
- J3, J4, J5, J7: footprint Connector_PinHeader_2.54mm:PinHeader_1x04_P2.54mm_Vertical -> Connector_JST:JST_XH_B4B-XH-A_1x04_P2.50mm_Vertical
- J6: footprint (none) -> Connector_PinHeader_2.54mm:PinHeader_1x05_P2.54mm_Vertical
Changed lines of the file:
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@@
 			)
 		)
-		(property "Footprint" "Connector_PinHeader_2.54mm:PinHeader_1x04_P2.54mm_Vertical"
+		(property "Footprint" "Connector_JST:JST_XH_B4B-XH-A_1x04_P2.50mm_Vertical"
 			(at 337.82 64.77 0)
 			(hide yes)
@@
 			)
 		)
-		(property "Footprint" "Connector_PinHeader_2.54mm:PinHeader_1x04_P2.54mm_Vertical"
+		(property "Footprint" "Connector_JST:JST_XH_B4B-XH-A_1x04_P2.50mm_Vertical"
 			(at 337.82 46.99 0)
 			(hide yes)
@@
 			)
 		)
-		(property "Footprint" ""
+		(property "Footprint" "Connector_PinHeader_2.54mm:PinHeader_1x05_P2.54mm_Vertical"
 			(at 337.82 85.09 0)
 			(hide yes)
@@
 			)
 		)
-		(property "Footprint" "Connector_PinHeader_2.54mm:PinHeader_1x04_P2.54mm_Vertical"
+		(property "Footprint" "Connector_JST:JST_XH_B4B-XH-A_1x04_P2.50mm_Vertical"
 			(at 369.57 64.77 0)
 			(hide yes)
@@
 			)
 		)
-		(property "Footprint" "Connector_PinHeader_2.54mm:PinHeader_1x04_P2.54mm_Vertical"
+		(property "Footprint" "Connector_JST:JST_XH_B4B-XH-A_1x04_P2.50mm_Vertical"
 			(at 369.57 46.99 0)
 			(hide yes)

Commit message: drafted pcb layout
Parts:
- added D2: D_Schottky, Diode_SMD:D_0402_1005Metric, symbol Device:D_Schottky
- added J10, J9: Conn_01x01, Connector_Wire:SolderWirePad_1x01_SMD_1x2mm, symbol Connector_Generic:Conn_01x01
- J3, J5, J7: footprint Connector_JST:JST_XH_B4B-XH-A_1x04_P2.50mm_Vertical -> Connector_PinHeader_2.54mm:PinHeader_1x04_P2.54mm_Vertical
- J4: footprint Connector_JST:JST_XH_B4B-XH-A_1x04_P2.50mm_Vertical -> Connector_PinSocket_2.54mm:PinSocket_1x04_P2.54mm_Vertical
- J8: footprint Connector_JST:JST_XH_B3B-XH-A_1x03_P2.50mm_Vertical -> Connector_PinHeader_2.54mm:PinHeader_1x03_P2.54mm_Vertical
- L1, L2: footprint Package_TO_SOT_SMD:SOT-583-8 -> Inductor_SMD:L_0805_2012Metric
Connections:
- net GND: now also J10.1 (Pin_1)
- net VBUS: now also D2.1 (K)
- new net: D2.2 (A), J9.1 (Pin_1)
Other:
- moved on the sheet: D3, D4, R20, R21

Commit message: routed mcu and power on pcb
Parts:
- C24, C25: footprint Capacitor_SMD:C_0402_1005Metric -> Capacitor_SMD:C_0603_1608Metric
- D1, D2: footprint Diode_SMD:D_0402_1005Metric -> Diode_SMD:D_SMA
Changed lines of the file:
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@@
 			)
 		)
-		(property "Footprint" "Capacitor_SMD:C_0402_1005Metric"
+		(property "Footprint" "Capacitor_SMD:C_0603_1608Metric"
 			(at 86.0552 107.95 0)
 			(hide yes)
@@
 			)
 		)
-		(property "Footprint" "Capacitor_SMD:C_0402_1005Metric"
+		(property "Footprint" "Capacitor_SMD:C_0603_1608Metric"
 			(at 42.8752 107.95 0)
 			(hide yes)
@@
 			)
 		)
-		(property "Footprint" "Diode_SMD:D_0402_1005Metric"
+		(property "Footprint" "Diode_SMD:D_SMA"
 			(at 73.66 30.48 0)
 			(hide yes)
@@
 			)
 		)
-		(property "Footprint" "Diode_SMD:D_0402_1005Metric"
+		(property "Footprint" "Diode_SMD:D_SMA"
 			(at 320.04 111.76 0)
 			(hide yes)

Commit message: finished routing pcb
Connections:
- net +3.3V is gone; now on net +3V3: J3.1 (Pin_1), J4.1 (Pin_1), J5.1 (Pin_1), J7.1 (Pin_1), R21.1
- net LMS_CS is gone; now on net LSM_CS: U1.33 (GPIO21)
- net BMP_INT: now also U1.27 (GPIO16)
- net LSM_INT1: now also U1.29 (GPIO18)
- net LSM_INT2: now also U1.35 (GPIO23)
- net MISO: no longer U3.14 (SDA)
- net MMC_INT: now also U1.19 (GPIO15)
- net MOSI: now also U3.14 (SDA)
- no-connect marks 9 -> 5

Commit message: fixed pin footprint
Parts:
- J4: footprint Connector_PinSocket_2.54mm:PinSocket_1x04_P2.54mm_Vertical -> Connector_PinHeader_2.54mm:PinHeader_1x04_P2.54mm_Vertical
Changed lines of the file:
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@@
 			)
 		)
-		(property "Footprint" "Connector_PinSocket_2.54mm:PinSocket_1x04_P2.54mm_Vertical"
+		(property "Footprint" "Connector_PinHeader_2.54mm:PinHeader_1x04_P2.54mm_Vertical"
 			(at 337.82 64.77 0)
 			(hide yes)

Commit message: added bom
Parts:
- C1, C2: MPN (none) -> CL05C330JB5NNNC
- C10, C26, C28, C29, C4: MPN (none) -> GRM155R60J475ME47D
- C11, C12, C13, C14, C15, C16, C17, C18, C22, C23, C5, C6, C7, C8, C9: MPN (none) -> GRM155R71H104KE14D
- C19: MPN (none) -> GRM188R61A106ME69D
- C20, C21: MPN (none) -> CL05A105KO5NNNC
- C24: MPN (none) -> GRM188R60J476ME15D
- C25: MPN (none) -> C1608X5R0J226M080AC
- D1, D2: MPN (none) -> SS210A
- D3: MPN (none) -> LTST-C190GKT
- D4: MPN (none) -> LTST-C190KRKT
- J1: MPN (none) -> UJ20-C-H-G-SMT-1-P16-TR
- J10, J3, J4, J5, J6, J7, J8, J9: now not fitted
- J2: MPN (none) -> MSD-7-A
- L1: MPN (none) -> DFE201210U-1R0M=P2
- L2: MPN (none) -> AOTA-B201610S3R3-101-T
- R1, R2: MPN (none) -> RC0402FR-075K1L
- R10, R11, R4, R6, R7, R8, R9: MPN (none) -> RC0402FR-0710KL
- R12: MPN (none) -> RC0402FR-13511KL
- R13: MPN (none) -> RK73H1ETTP9102F
- R14, R16: MPN (none) -> RC0402FR-07100KL
- R15: MPN (none) -> RC0402FR-0733RL
- R17: MPN (none) -> CPF0402B150KE1
- R18, R19: MPN (none) -> RK73H1ETTP4701F
- R20, R21, R3, R5: MPN (none) -> ERJ-2RKF1001X
- SW1: MPN (none) -> SKRKAEE020
- U1: MPN (none) -> RP2350A
- U2: MPN (none) -> MMC5983MA
- U3: MPN (none) -> LSM6DSMTR
- U4: MPN (none) -> BMP384
- U5: MPN (none) -> TPS631000DRLR
- U6: MPN (none) -> W25Q128JVSIQ TR
- Y1: value ABM8-272-T3 -> 12MHz; MPN (none) -> ABM8-272-T3

Commit message: updated readme
Parts:
- J10, J3, J4, J5, J6, J7, J8, J9: now fitted
Changed lines of the file:
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@@
 		(on_board yes)
 		(in_pos_files yes)
-		(dnp yes)
+		(dnp no)
 		(property "Reference" "J4"
 			(at 337.82 56.642 0)
@@
 		(on_board yes)
 		(in_pos_files yes)
-		(dnp yes)
+		(dnp no)
 		(property "Reference" "J3"
 			(at 337.82 38.862 0)
@@
 		(on_board yes)
 		(in_pos_files yes)
-		(dnp yes)
+		(dnp no)
 		(property "Reference" "J6"
 			(at 336.55 74.93 0)
@@
 		(on_board yes)
 		(in_pos_files yes)
-		(dnp yes)
+		(dnp no)
 		(property "Reference" "J7"
 			(at 369.57 56.642 0)
@@
 		(on_board yes)
 		(in_pos_files yes)
-		(dnp yes)
+		(dnp no)
 		(property "Reference" "J5"
 			(at 369.57 38.862 0)
@@
 		(on_board yes)
 		(in_pos_files yes)
-		(dnp yes)
+		(dnp no)
 		(fields_autoplaced yes)
 		(property "Reference" "J9"
@@
 		(on_board yes)
 		(in_pos_files yes)
-		(dnp yes)
+		(dnp no)
 		(property "Reference" "J8"
 			(at 368.3 74.676 0)
@@
 		(on_board yes)
 		(in_pos_files yes)
-		(dnp yes)
+		(dnp no)
 		(fields_autoplaced yes)
 		(property "Reference" "J10"
